File: Hardware/Ink-Board.brd (EAGLE design)
At the start: 46 x 35 mm, 105 parts, among them IC1 BQ25180YBGR, IC2 DRV2605YZFR, IC3 BMA423, IC9 RT6160AWSC, J1 503480-2400, J2 TC2030-IDC, J4 KH-TYPE-C-16P, Q1 20V/4.2A/52mΩ/1.4W, Q3 SI1308EDL-T1-GE3, U3 MAX17048G+T10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

Commit message: Updating the project
Routing:
- net GND: track 375.3 -> 403.1 mm, vias 25 -> 28
- net SDA/1.4C: track 0.02 -> 20.5 mm, vias 0 -> 2
- net IMU_INT2: track 0.00 -> 20.0 mm, vias 0 -> 2
- net PMIC_INT: track 0.00 -> 15.5 mm, vias 0 -> 2
- net 3V3/2.4A: track 124.0 -> 139.5 mm, vias 13 -> 14
- net SCL/2.4C: track 24.8 -> 36.0 mm
- net RESET: track 19.3 -> 29.4 mm
- net DEC4_6: track 9.53 -> 18.1 mm, vias 0 -> 2
- net P0.14/1.5D: track 8.41 -> 16.9 mm
- net SWDCLK: track 20.7 -> 27.7 mm
- net VBAT/1.2A: track 7.95 -> 12.9 mm, vias 2 -> 4
- net VREG: track 38.8 -> 34.3 mm, vias 4 -> 3
- net N$35: track 4.57 -> 7.82 mm
- net N$26: track 12.7 -> 15.7 mm
- net RESE: track 26.4 -> 29.1 mm
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- added copper zone on layer 1, net GND
